Commit message: added slam mapping

File: imprimis_ws/src/imprimis/description/camera.xacro (robot description, xacro)
@@ -2,7 +2,7 @@
 <robot xmlns:xacro="http://www.ros.org/wiki/xacro" >
     <joint name="camera_joint" type="fixed">
-        <parent link="base_link"/>
+        <parent link="chassis"/>
         <child link="camera_link"/>
-        <origin xyz="${(base_length/2)} 0 ${(base_height/2-wheel_zoff)}" rpy="0 0 0"/>
+        <origin xyz="${base_length+0.01} 0 0.08" rpy="0 0 0"/>
     </joint>
     <link name="camera_link">

File: imprimis_ws/src/imprimis/description/gazebo_control.xacro (robot description, xacro)
@@ -1,11 +1,14 @@
 <?xml version="1.0"?>
 <robot xmlns:xacro="http://www.ros.org/wiki/xacro">
+<xacro:property name="base_width" value="0.62" />
+<xacro:property name="wheel_radius" value="0.17" />
+<xacro:property name="wheel_yoff" value="0.13"/>
     <gazebo>
         <plugin name='diff_drive' filename='libgazebo_ros_diff_drive.so'>
             <!-- Wheel Information -->
-            <left_joint>drivewhl_l_joint</left_joint>
-            <right_joint>drivewhl_r_joint</right_joint>
-            <wheel_separation>0.65</wheel_separation>
-            <wheel_diameter>0.254</wheel_diameter>
+            <left_joint>left_wheel_joint</left_joint>
+            <right_joint>right_wheel_joint</right_joint>
+            <wheel_separation>${base_width+(2*wheel_yoff)}</wheel_separation>
+            <wheel_diameter>${wheel_radius*2}</wheel_diameter>
             <!-- Limits -->
             <max_wheel_torque>200</max_wheel_torque>
@@ -17,4 +20,6 @@
             <publish_odom_tf>true</publish_odom_tf>
             <publish_wheel_tf>true</publish_wheel_tf>
+    <!-- <odometry_frame>odom</odometry_frame> -->
+    <!-- <robot_base_frame>base_link</robot_base_frame> -->
         </plugin>
     </gazebo>

File: imprimis_ws/src/imprimis/description/lidar.xacro (robot description, xacro)
@@ -1,23 +1,23 @@
 <?xml version="1.0"?>
-<robot xmlns:xacro="http://www.ros.org/wiki/xacro">
+<robot xmlns:xacro="http://www.ros.org/wiki/xacro" >
     <joint name="laser_joint" type="fixed">
-        <parent link="base_link" />
-        <child link="laser_frame" />
-        <origin xyz="0.1 0 0.175" rpy="0 0 0" />
+        <parent link="base_link"/>
+        <child link="laser_frame"/>
+          <origin xyz="0 0 ${base_height+0.02}" rpy="0 0 0"/>
     </joint>
     <link name="laser_frame">
         <visual>
             <geometry>
-                <cylinder radius="0.05" length="0.04" />
+                <cylinder radius="0.05" length="0.04"/>
             </geometry>
-            <material name="red" />
+            <material name="red"/>
         </visual>
         <collision>
             <geometry>
-                <cylinder radius="0.05" length="0.04" />
+                <cylinder radius="0.05" length="0.04"/>
             </geometry>
         </collision>
         <xacro:inertial_cylinder mass="0.1" length="0.04" radius="0.05">
-            <origin xyz="0 0 0" rpy="0 0 0" />
+            <origin xyz="0 0 0" rpy="0 0 0"/>
         </xacro:inertial_cylinder>
     </link>
@@ -26,5 +26,5 @@
         <sensor name="laser" type="ray">
             <pose> 0 0 0 0 0 0 </pose>
-            <visualize>false</visualize>
+            <visualize>true</visualize>
             <update_rate>10</update_rate>
             <ray>

File: imprimis_ws/src/imprimis/description/robot.urdf.xacro (robot description, xacro)
@@ -1,7 +1,9 @@
 <?xml version="1.0"?>
 <robot xmlns:xacro="http://www.ros.org/wiki/xacro"  name="robot">
-    <xacro:include filename="robot_core.xacro" />
-    <xacro:include filename="gazebo_control.xacro" />
-    <xacro:include filename="lidar.xacro" />
-    <xacro:include filename="camera.xacro" />
+	<xacro:include filename="robot_core.xacro" />
+	<!-- <xacro:include filename="ros2_control.xacro" /> -->
+	<xacro:include filename="gazebo_control.xacro" />
+	<xacro:include filename="lidar.xacro" />
+	<xacro:include filename="camera.xacro" />
+	<xacro:include filename="imu.xacro" />
 </robot>

File: imprimis_ws/src/imprimis/description/robot_core.xacro (robot description, xacro)
@@ -1,150 +1,137 @@
 <?xml version="1.0"?>
 <robot xmlns:xacro="http://www.ros.org/wiki/xacro">
-    <xacro:include filename="inertial_macros.xacro" />
-    <xacro:property name="base_width" value="0.61" />
-    <xacro:property name="base_length" value="0.92" />
-    <xacro:property name="base_height" value="0.3" />
-    <xacro:property name="wheel_radius" value="0.127" />
-    <xacro:property name="wheel_width" value="0.04" />
-    <xacro:property name="wheel_ygap" value="0.02" />
-    <xacro:property name="wheel_zoff" value="0.1" />
-    <xacro:property name="wheel_xoff" value="0.2" />
-    <xacro:property name="caster_xoff" value="0.24" />
-    <!-- Define intertial property macros  -->
-    <xacro:macro name="box_inertia" params="m w h d">
-        <inertial>
-            <origin xyz="0 0 0" rpy="${pi/2} 0 ${pi/2}" />
-            <mass value="${m}" />
-            <inertia ixx="${(m/12) * (h*h + d*d)}" ixy="0.0" ixz="0.0" iyy="${(m/12) * (w*w + d*d)}"
-                iyz="0.0" izz="${(m/12) * (w*w + h*h)}" />
-        </inertial>
-    </xacro:macro>
-    <xacro:macro name="cylinder_inertia" params="m r h">
-        <inertial>
-            <origin xyz="0 0 0" rpy="${pi/2} 0 0" />
-            <mass value="${m}" />
-            <inertia ixx="${(m/12) * (3*r*r + h*h)}" ixy="0" ixz="0" iyy="${(m/12) * (3*r*r + h*h)}"
-                iyz="0" izz="${(m/2) * (r*r)}" />
-        </inertial>
-    </xacro:macro>
-    <xacro:macro name="sphere_inertia" params="m r">
-        <inertial>
-            <mass value="${m}" />
-            <inertia ixx="${(2/5) * m * (r*r)}" ixy="0.0" ixz="0.0" iyy="${(2/5) * m * (r*r)}"
-                iyz="0.0" izz="${(2/5) * m * (r*r)}" />
-        </inertial>
-    </xacro:macro>
-    <!-- Robot Base -->
-    <link name="base_link">
-        <visual>
-            <geometry>
-                <box size="${base_length} ${base_width} ${base_height}" />
-            </geometry>
-            <material name="Cyan">
-                <color rgba="0 1.0 1.0 1.0" />
-            </material>
-        </visual>
-        <collision>
-            <geometry>
-                <box size="${base_length} ${base_width} ${base_height}" />
-            </geometry>
-        </collision>
-        <xacro:box_inertia m="15" w="${base_width}" d="${base_length}" h="${base_height}" />
-    </link>
-    <!-- Robot Footprint -->
-    <link name="base_footprint" />
-    <joint name="base_joint" type="fixed">
-        <parent link="base_link" />
-        <child link="base_footprint" />
-        <origin xyz="0.0 0.0 ${-(wheel_radius+wheel_zoff)}" rpy="0 0 0" />
-    </joint>
-    <!-- Wheels -->
-    <xacro:macro name="wheel" params="prefix x_reflect y_reflect">
-        <link name="${prefix}_link">
-            <visual>
-                <origin xyz="0 0 0" rpy="${pi/2} 0 0" />
-                <geometry>
-                    <cylinder radius="${wheel_radius}" length="${wheel_width}" />
-                </geometry>
-                <material name="Gray">
-                    <color rgba="0.5 0.5 0.5 1.0" />
-                </material>
-            </visual>
-            <collision>
-                <origin xyz="0 0 0" rpy="${pi/2} 0 0" />
-                <geometry>
-                    <cylinder radius="${wheel_radius}" length="${wheel_width}" />
-                </geometry>
-            </collision>
-            <xacro:cylinder_inertia m="0.5" r="${wheel_radius}" h="${wheel_width}" />
-        </link>
-        <gazebo reference="${prefix}_link">
-            <material>Gazebo/Black</material>
-        </gazebo>
-        <joint name="${prefix}_joint" type="continuous">
-            <parent link="base_link" />
-            <child link="${prefix}_link" />
-            <origin
-                xyz="${x_reflect*wheel_xoff} ${y_reflect*(base_width/2+wheel_ygap)} ${-wheel_zoff}"
-                rpy="0 0 0" />
-            <axis xyz="0 1 0" />
-        </joint>
-    </xacro:macro>
-    <xacro:wheel prefix="drivewhl_l" x_reflect="-1" y_reflect="1" />
-    <xacro:wheel prefix="drivewhl_r" x_reflect="-1" y_reflect="-1" />
-    <!-- Caster Wheel -->
-    <link name="front_r_caster">
-        <visual>
-            <geometry>
-                <sphere radius="${(wheel_radius+wheel_zoff-(base_height/2))}" />
-            </geometry>
-            <material name="Cyan">
-                <color rgba="0 1.0 1.0 1.0" />
-            </material>
-        </visual>
-        <collision>
-            <origin xyz="0 0 0" rpy="0 0 0" />
-            <geometry>
-                <sphere radius="${(wheel_radius+wheel_zoff-(base_height/2))}" />
-            </geometry>
-        </collision>
-        <xacro:sphere_inertia m="0.5" r="${(wheel_radius+wheel_zoff-(base_height/2))}" />
-    </link>
-    <gazebo reference="front_r_caster">
-        <material>Gazebo/Black</material>
-        <mu1 value="0.001"/>
-        <mu2 value="0.001"/>
-    </gazebo>
-    <joint name="caster_r_joint" type="fixed">
-        <parent link="base_link" />
-        <child link="front_r_caster" />
-        <origin xyz="${caster_xoff} 0.14 ${-(base_height/2)}" rpy="0 0 0" />
-    </joint>
-    <link name="front_l_caster">
-        <visual>
-            <geometry>
-                <sphere radius="${(wheel_radius+wheel_zoff-(base_height/2))}" />
-            </geometry>
-            <material name="Cyan">
-                <color rgba="0 1.0 1.0 1.0" />
-            </material>
-        </visual>
-        <collision>
-            <origin xyz="0 0 0" rpy="0 0 0" />
-            <geometry>
-                <sphere radius="${(wheel_radius+wheel_zoff-(base_height/2))}" />
-            </geometry>
-        </collision>
-        <xacro:sphere_inertia m="0.5" r="${(wheel_radius+wheel_zoff-(base_height/2))}" />
-    </link>
-    <gazebo reference="front_l_caster">
-        <material>Gazebo/Black</material>
-        <mu1 value="0.001"/>
-        <mu2 value="0.001"/>
-    </gazebo>
-    <joint name="caster_l_joint" type="fixed">
-        <parent link="base_link" />
-        <child link="front_l_caster" />
-        <origin xyz="${caster_xoff} -0.14 ${-(base_height/2)}" rpy="0 0 0" />
-    </joint>
+<material name="white">
+    <color rgba="1 1 1 1"/>
+</material>
+<material name="orange">
+    <color rgba="1 0.3 0.1 1"/>
+</material>
+<material name="blue">
+    <color rgba="0.2 0.2 1 1"/>
+</material>
+<material name="black">
+    <color rgba="0 0 0 1"/>
+</material>
+<xacro:include filename="inertial_macros.xacro" />
+<xacro:property name="base_width" value="0.62" />
+<xacro:property name="base_length" value="1.02" />
+<xacro:property name="base_height" value="0.51" />
+<xacro:property name="wheel_radius" value="0.17" />
+<xacro:property name="wheel_width" value="0.1" />
+<xacro:property name="wheel_yoff" value="0.13"/>
+<xacro:property name="wheel_zoff" value="0.054"/>
+<link name="base_link">
+</link>
+  <joint name="base_footprint_joint" type="fixed">
+    <parent link="base_link"/>
+    <child link="base_footprint"/>
+    <origin xyz="0 0 0" rpy="0 0 0"/>
+  </joint>
+<link name="base_footprint">
+</link>
+<joint name="chassis_joint" type="fixed">
+    <parent link="base_link"/>
+    <child link="chassis"/>
+    <origin xyz="-0.85 0 0"/>
+</joint>
+<link name="chassis">
+    <visual>
+        <origin xyz="${base_length/2} 0 ${base_height/2}" rpy="0 0 0"/>
+        <geometry>
+            <box size="${base_length} ${base_width} ${base_height}" />
+        </geometry>
+        <material name="white"/>
+    </visual>
+    <collision>
+        <origin xyz="${base_length/2} 0 ${base_height/2}" rpy="0 0 0"/>
+        <geometry>
+            <box size="${base_length} ${base_width} ${base_height}" />
+        </geometry>
+    </collision>
+	<xacro:inertial_box mass="0.5" x="${base_length}" y="${base_width}" z="${base_height}">
+        <origin xyz="${base_length/2} 0 ${base_height/2}" rpy="0 0 0"/>
+	</xacro:inertial_box>
+</link>
+<gazebo reference="chassis">
+    <material>Gazebo/White</material>
+</gazebo>
+<!-- LEFT WHEEL -->
+<joint name="left_wheel_joint" type="continuous">
+    <parent link="base_link"/>
+    <child link="left_wheel"/>
+    <origin xyz="0 ${base_width/2+wheel_yoff} ${wheel_zoff}" rpy="-${pi/2} 0 0"/>
+    <axis xyz="0 0 1"/>
+</joint>
+<link name="left_wheel">
+    <visual>
+        <geometry>
+            <cylinder length="${wheel_width}" radius="${wheel_radius}" />
+        </geometry>
+        <material name="blue"/>
+    </visual>
+    <collision>
+        <geometry>
+            <cylinder length="${wheel_width}" radius="${wheel_radius}" />
+        </geometry>
+    </collision>
+    <xacro:inertial_cylinder mass="0.1" length="${wheel_width}" radius="${wheel_radius}">
+        <origin xyz="0 0 0" rpy="0 0 0"/>
+    </xacro:inertial_cylinder>
+</link>
+<gazebo reference="left_wheel">
+    <material>Gazebo/Blue</material>
+</gazebo>
+<!-- RIGHT WHEEL -->
+<joint name="right_wheel_joint" type="continuous">
+    <parent link="base_link"/>
+    <child link="right_wheel"/>
+    <origin xyz="0 ${-(base_width/2+wheel_yoff)} ${wheel_zoff}" rpy="${pi/2} 0 0"/>
+    <axis xyz="0 0 -1"/>
+</joint>
+<link name="right_wheel">
+    <visual>
+        <geometry>
+            <cylinder length="${wheel_width}" radius="${wheel_radius}" />
+        </geometry>
+        <material name="blue"/>
+    </visual>
+    <collision>
+        <geometry>
+            <cylinder length="${wheel_width}" radius="${wheel_radius}" />
+        </geometry>
+    </collision>
+        <xacro:inertial_cylinder mass="0.1" length="${wheel_width}" radius="${wheel_radius}">
+        <origin xyz="0 0 0" rpy="0 0 0"/>
+    </xacro:inertial_cylinder>
+</link>
+<gazebo reference="right_wheel">
+    <material>Gazebo/Blue</material>
+</gazebo>
+<!-- CASTER WHEEL -->
+<joint name="caster_wheel_joint" type="fixed">
+    <parent link="chassis"/>
+    <child link="caster_wheel"/>
+    <origin xyz="0.15 0 ${wheel_zoff}" rpy="0 0 0"/>
+</joint>
+<link name="caster_wheel">
+    <visual>
+        <geometry>
+            <sphere radius="${wheel_radius}" />
+        </geometry>
+        <material name="black"/>
+    </visual>
+    <collision>
+        <geometry>
+            <sphere radius="${wheel_radius}" />
+        </geometry>
+    </collision>
+    <xacro:inertial_sphere mass="0.1" radius="${wheel_radius}">
+        <origin xyz="0 0 0" rpy="0 0 0"/>
+    </xacro:inertial_sphere>
+</link>
+<gazebo reference="caster_wheel">
+    <material>Gazebo/Black</material>
+    <mu1 value="0.001"/>
+    <mu2 value="0.001"/>
+</gazebo>
 </robot>
