Commit message: Updated gazebo sim to work with ros2_control

File: imprimis_ws/src/imprimis/description/robot.urdf.xacro (robot description, xacro)
@@ -2,6 +2,6 @@
 <robot xmlns:xacro="http://www.ros.org/wiki/xacro"  name="robot">
 	<xacro:include filename="robot_core.xacro" />
-	<!-- <xacro:include filename="ros2_control.xacro" /> -->
-	<xacro:include filename="gazebo_control.xacro" />
+<!--	<xacro:include filename="gazebo_control.xacro" /> -->
+	<xacro:include filename="ros2_control.xacro" />
 	<xacro:include filename="lidar.xacro" />
 	<xacro:include filename="camera.xacro" />

File: imprimis_ws/src/imprimis/description/robot_core.xacro (robot description, xacro)
@@ -17,5 +17,5 @@
 <xacro:property name="base_length" value="1.02" />
 <xacro:property name="base_height" value="0.51" />
-<xacro:property name="wheel_radius" value="0.17" />
+<xacro:property name="wheel_radius" value="0.165" />
 <xacro:property name="wheel_width" value="0.1" />
 <xacro:property name="wheel_yoff" value="0.13"/>

File: imprimis_ws/src/imprimis/description/ros2_control.xacro (robot description, xacro)
@@ -24,5 +24,5 @@
 <gazebo>
     <plugin filename="libgazebo_ros2_control.so" name="gazebo_ros2_control">
-        <parameters>/home/hyperlabs/Desktop/imprimis/imprimis_ws/src/imprimis/config/my_controllers.yaml</parameters>
+        <parameters>$(find imprimis)/config/my_controllers.yaml</parameters>
     </plugin>
 </gazebo>
