Commit message: Replaced example URDF with prototype imprimis URDF. Added cmd_vel_gui package

File: imprimis_ws/src/ros2_control_demo_example_2/description/urdf/diffbot_description.urdf.xacro (robot description, xacro)
@@ -1,54 +1,93 @@
 <?xml version="1.0"?>
 <robot xmlns:xacro="http://www.ros.org/wiki/xacro">
-  <xacro:macro name="diffbot" params="prefix">
-  <!-- Constants for robot dimensions -->
-  <xacro:property name="PI" value="3.1415926535897931"/>
-  <xacro:property name="base_mass" value="0.3" /> <!-- arbitrary value for base mass -->
-  <xacro:property name="base_width" value="0.1" />
-  <xacro:property name="base_length" value="0.1" />
-  <xacro:property name="base_height" value="0.05" />
-  <xacro:property name="wheel_mass" value="0.3" /> <!-- arbitrary value for wheel mass -->
-  <xacro:property name="wheel_len" value="0.020" />
-  <xacro:property name="wheel_radius" value="0.015" />
-  <xacro:property name="caster_wheel_mass" value="0.1" /> <!-- arbitrary value for caster wheel mass -->
-  <xacro:property name="caster_wheel_radius" value="0.015" />
-  <xacro:property name="z_offset" value="-${base_height/2}" /> <!-- Space btw top of beam and the each joint -->
-  <xacro:include filename="inertial_macros.xacro" />
-  <!-- Base Link -->
-  <link name="${prefix}base_link">
-    <collision>
-      <origin xyz="0 0 0" rpy="0 0 0"/>
-      <geometry>
-        <box size="${base_width} ${base_length} ${base_height}"/>
-      </geometry>
-    </collision>
-    <visual>
-      <origin xyz="0 0 ${base_height/2}" rpy="0 0 0"/>
-      <geometry>
-        <box size="${base_width} ${base_length} ${base_height}"/>
-      </geometry>
-      <material name="orange"/>
-    </visual>
-    <inertial>
-      <origin xyz="0 0 0" rpy="0 0 0"/>
-      <mass value="${base_mass}"/>
-      <inertia
-        ixx="${base_mass / 12.0 * (base_length*base_length + base_height*base_height)}" ixy="0.0" ixz="0.0"
-        iyy="${base_mass / 12.0 * (base_height*base_height + base_width*base_width)}" iyz="0.0"
-        izz="${base_mass / 12.0 * (base_width*base_width + base_length*base_length)}"/>
-      </inertial>
-    </link>
-    <joint name="${prefix}left_wheel_joint" type="continuous">
+<xacro:macro name="diffbot" params="prefix">
+<!-- Constants for robot dimensions -->
+<xacro:property name="PI" value="3.1415926535897931"/>
+<!-- Constants for robot dimensions -->
+<xacro:property name="base_mass" value="0.3" />
+<xacro:property name="wheel_mass" value="0.3" />
+<xacro:property name="base_width" value="0.62" />
+<xacro:property name="base_length" value="1.016" />
+<xacro:property name="base_height" value="0.51" />
+<xacro:property name="wheel_len" value="0.1" />
+<xacro:property name="wheel_radius" value="0.165" />
+<xacro:property name="wheel_yoff" value="0.13"/>
+<xacro:property name="wheel_zoff" value="0.054"/>
+<xacro:property name="base_top_width" value="0.749"/>
+<xacro:property name="base_top_height" value="0.305"/>
+<xacro:include filename="inertial_macros.xacro" />
+<link name="${prefix}base_link">
+</link>
+<joint name="base_footprint_joint" type="fixed">
+  <parent link="base_link"/>
+  <child link="base_footprint"/>
+  <origin xyz="-0.35 0 ${-wheel_radius+wheel_zoff}"/>
+</joint>
+<link name="base_footprint">
+</link>
+<joint name="${prefix}chassis_joint" type="fixed">
+  <parent link="${prefix}base_link"/>
+  <child link="${prefix}chassis"/>
+  <origin xyz="-0.85 0 0"/>
+</joint>
+<link name="${prefix}chassis">
+  <visual>
+    <origin xyz="${base_length/2} 0 ${base_height/2}" rpy="0 0 0"/>
+    <geometry>
+    <box size="${base_length} ${base_width} ${base_height}" />
+    </geometry>
+    <material name="white"/>
+  </visual>
+  <collision>
+    <origin xyz="${base_length/2} 0 ${base_height/2}" rpy="0 0 0"/>
+    <geometry>
+    <box size="${base_length} ${base_width} ${base_height}" />
+    </geometry>
+  </collision>
+  <xacro:inertial_box mass="0.5" x="${base_length}" y="${base_width}" z="${base_height}"> <!-- inertial macro -->
+    <origin xyz="${base_length/2} 0 ${base_height/2}" rpy="0 0 0"/>
+  </xacro:inertial_box>
+</link>
+<joint name="${prefix}left_wheel_joint" type="continuous">
+  <parent link="${prefix}base_link"/>
+  <child link="${prefix}left_wheel"/>
+  <origin xyz="0 ${base_width/2+wheel_yoff} ${wheel_zoff}" rpy="-${pi/2} 0 0"/>
+  <axis xyz="0 0 1"/>
+  <dynamics damping="0.2"/>
+</joint>
+    <!-- left wheel Link -->
+<link name="${prefix}left_wheel">
+  <collision>
+    <origin xyz="0 0 0"/>
+    <geometry>
+      <cylinder length="${wheel_len}" radius="${wheel_radius}"/>
+    </geometry>
+  </collision>
+  <visual>
+    <origin xyz="0 0 0"/>
+    <geometry>
+      <cylinder length="${wheel_len}" radius="${wheel_radius}"/>
+    </geometry>
+    <material name="black"/>
+  </visual>
+  <inertial>
+    <origin xyz="0 0 0" rpy="${PI/2} 0 0"/>
+    <mass value="${wheel_mass}"/>
+    <inertia
+      ixx="${wheel_mass / 12.0 * (3*wheel_radius*wheel_radius + wheel_len*wheel_len)}" ixy="0.0" ixz="0.0"
+      iyy="${wheel_mass / 12.0 * (3*wheel_radius*wheel_radius + wheel_len*wheel_len)}" iyz="0.0"
+      izz="${wheel_mass / 2.0 * wheel_radius*wheel_radius}"/>
+    </inertial>
+  </link>
+    <joint name="${prefix}right_wheel_joint" type="continuous">
       <parent link="${prefix}base_link"/>
-      <child link="${prefix}left_wheel"/>
-      <origin xyz="0 -${base_width/2} ${z_offset}" rpy="0 0 0"/>
-      <axis xyz="0 1 0"/>
-      <dynamics damping="0.2"/>
-      <limit effort="100" velocity="1.0"/>
+      <child link="${prefix}right_wheel"/>
+      <origin xyz="0 ${-(base_width/2+wheel_yoff)} ${wheel_zoff}" rpy="${pi/2} 0 0"/>
+      <axis xyz="0 0 -1"/>
+      <dynamics damping="0.1"/>
     </joint>
-    <!-- left wheel Link -->
-    <link name="${prefix}left_wheel">
+    <!-- right wheel Link -->
+    <link name="${prefix}right_wheel">
       <collision>
-        <origin xyz="0 0 0" rpy="${PI/2} 0 0"/>
         <geometry>
           <cylinder length="${wheel_len}" radius="${wheel_radius}"/>
@@ -56,5 +95,4 @@
       </collision>
       <visual>
-        <origin xyz="0 0 0" rpy="${PI/2} 0 0"/>
         <geometry>
           <cylinder length="${wheel_len}" radius="${wheel_radius}"/>
@@ -69,95 +107,5 @@
           iyy="${wheel_mass / 12.0 * (3*wheel_radius*wheel_radius + wheel_len*wheel_len)}" iyz="0.0"
           izz="${wheel_mass / 2.0 * wheel_radius*wheel_radius}"/>
-        </inertial>
-      </link>
-    <joint name="${prefix}right_wheel_joint" type="continuous">
-      <parent link="${prefix}base_link"/>
-      <child link="${prefix}right_wheel"/>
-      <origin xyz="0 ${base_width/2} ${z_offset}" rpy="0 0 0"/>
-      <axis xyz="0 1 0"/>
-      <dynamics damping="0.2"/>
-      <limit effort="100" velocity="1.0"/>
-    </joint>
-    <!-- right wheel Link -->
-    <link name="${prefix}right_wheel">
-      <collision>
-        <origin xyz="0 0 0" rpy="${PI/2} 0 0"/>
-        <geometry>
-          <cylinder length="${wheel_len}" radius="${wheel_radius}"/>
-        </geometry>
-      </collision>
-      <visual>
-        <origin xyz="0 0 0" rpy="${PI/2} 0 0"/>
-        <geometry>
-          <cylinder length="${wheel_len}" radius="${wheel_radius}"/>
-        </geometry>
-        <material name="black"/>
-      </visual>
-      <inertial>
-        <origin xyz="0 0 0" rpy="${PI/2} 0 0"/>
-        <mass value="${wheel_mass}"/>
-        <inertia
-          ixx="${wheel_mass / 12.0 * (3*wheel_radius*wheel_radius + wheel_len*wheel_len)}" ixy="0.0" ixz="0.0"
-          iyy="${wheel_mass / 12.0 * (3*wheel_radius*wheel_radius + wheel_len*wheel_len)}" iyz="0.0"
-          izz="${wheel_mass / 2.0 * wheel_radius*wheel_radius}"/>
-        </inertial>
-      </link>
-    <joint name="${prefix}caster_frontal_wheel_joint" type="fixed">
-      <parent link="${prefix}base_link"/>
-      <child link="${prefix}caster_frontal_wheel"/>
-      <origin xyz="${base_width/2 - caster_wheel_radius} 0 ${z_offset}" rpy="0 0 0"/>
-    </joint>
-    <!-- caster frontal wheel Link -->
-    <link name="${prefix}caster_frontal_wheel">
-      <collision>
-        <origin xyz="0 0 0" rpy="0 0 0"/>
-        <geometry>
-          <sphere radius="${caster_wheel_radius}"/>
-        </geometry>
-      </collision>
-      <visual>
-        <origin xyz="0 0 0" rpy="0 0 0"/>
-        <geometry>
-          <sphere radius="${caster_wheel_radius}"/>
-        </geometry>
-        <material name="white"/>
-      </visual>
-      <inertial>
-        <origin xyz="0 0 0" rpy="0 0 0"/>
-        <mass value="${caster_wheel_mass}"/>
-        <inertia
-          ixx="${caster_wheel_mass * 0.4 * (caster_wheel_radius * caster_wheel_radius)}" ixy="0.0" ixz="0.0"
-          iyy="${caster_wheel_mass * 0.4 * (caster_wheel_radius * caster_wheel_radius)}" iyz="0.0"
-          izz="${caster_wheel_mass * 0.4 * (caster_wheel_radius * caster_wheel_radius)}"/>
-        </inertial>
-      </link>
-    <joint name="${prefix}caster_rear_wheel_joint" type="fixed">
-      <parent link="${prefix}base_link"/>
-      <child link="${prefix}caster_rear_wheel"/>
-      <origin xyz="${-base_width/2 + caster_wheel_radius} 0 ${z_offset}" rpy="0 0 0"/>
-    </joint>
-    <!-- caster rear wheel Link -->
-    <link name="${prefix}caster_rear_wheel">
-      <collision>
-        <origin xyz="0 0 0" rpy="0 0 0"/>
-        <geometry>
-          <sphere radius="${caster_wheel_radius}"/>
-        </geometry>
-      </collision>
-      <visual>
-        <origin xyz="0 0 0" rpy="0 0 0"/>
-        <geometry>
-          <sphere radius="${caster_wheel_radius}"/>
-        </geometry>
-        <material name="white"/>
-      </visual>
-      <inertial>
-        <origin xyz="0 0 0" rpy="0 0 0"/>
-        <mass value="${caster_wheel_mass}"/>
-        <inertia
-          ixx="${caster_wheel_mass * 0.4 * (caster_wheel_radius * caster_wheel_radius)}" ixy="0.0" ixz="0.0"
-          iyy="${caster_wheel_mass * 0.4 * (caster_wheel_radius * caster_wheel_radius)}" iyz="0.0"
-          izz="${caster_wheel_mass * 0.4 * (caster_wheel_radius * caster_wheel_radius)}"/>
-        </inertial>
+        </inertial> <!-- for some reason, the inertial cylinder macro was not parsing -->
       </link>
   </xacro:macro>
