Commit message: Renamed description package to imprimis_description

File: imprimis_ws/src/imprimis_description/urdf/diffbot.ros2_control.xacro (robot description, xacro)
@@ -1,5 +1,5 @@
 <?xml version="1.0"?>
 <robot xmlns:xacro="http://www.ros.org/wiki/xacro">
-  <xacro:macro name="diffbot_ros2_control" params="name prefix use_mock_hardware">
+  <xacro:macro name="diffbot_ros2_control" params="name use_mock_hardware">
     <ros2_control name="${name}" type="system">
       <xacro:unless value="${use_mock_hardware}">
@@ -16,10 +16,10 @@
         </hardware>
       </xacro:if>
-      <joint name="${prefix}left_wheel_joint">
+      <joint name="left_wheel_joint">
         <command_interface name="velocity"/>
         <state_interface name="position"/>
         <state_interface name="velocity"/>
       </joint>
-      <joint name="${prefix}right_wheel_joint">
+      <joint name="right_wheel_joint">
         <command_interface name="velocity"/>
         <state_interface name="position"/>

File: imprimis_ws/src/imprimis_description/urdf/diffbot_description.urdf.xacro (robot description, xacro)
@@ -1,5 +1,5 @@
 <?xml version="1.0"?>
 <robot xmlns:xacro="http://www.ros.org/wiki/xacro">
-<xacro:macro name="diffbot" params="prefix">
+<xacro:macro name="diffbot">
 <!-- Constants for robot dimensions -->
 <xacro:property name="PI" value="3.1415926535897931"/>
@@ -17,5 +17,5 @@
 <xacro:property name="base_top_height" value="0.305"/>
 <xacro:include filename="inertial_macros.xacro" />
-<link name="${prefix}base_link">
+<link name="base_link">
 </link>
 <joint name="base_footprint_joint" type="fixed">
@@ -26,10 +26,10 @@
 <link name="base_footprint">
 </link>
-<joint name="${prefix}chassis_joint" type="fixed">
-  <parent link="${prefix}base_link"/>
-  <child link="${prefix}chassis"/>
+<joint name="chassis_joint" type="fixed">
+  <parent link="base_link"/>
+  <child link="chassis"/>
   <origin xyz="-0.85 0 0"/>
 </joint>
-<link name="${prefix}chassis">
+<link name="chassis">
   <visual>
     <origin xyz="${base_length/2} 0 ${base_height/2}" rpy="0 0 0"/>
@@ -49,7 +49,7 @@
   </xacro:inertial_box>
 </link>
-<joint name="${prefix}left_wheel_joint" type="continuous">
-  <parent link="${prefix}base_link"/>
-  <child link="${prefix}left_wheel"/>
+<joint name="left_wheel_joint" type="continuous">
+  <parent link="base_link"/>
+  <child link="left_wheel"/>
   <origin xyz="0 ${base_width/2+wheel_yoff} ${wheel_zoff}" rpy="-${pi/2} 0 0"/>
   <axis xyz="0 0 1"/>
@@ -57,5 +57,5 @@
 </joint>
     <!-- left wheel Link -->
-<link name="${prefix}left_wheel">
+<link name="left_wheel">
   <collision>
     <origin xyz="0 0 0"/>
@@ -80,7 +80,7 @@
     </inertial>
   </link>
-    <joint name="${prefix}right_wheel_joint" type="continuous">
-      <parent link="${prefix}base_link"/>
-      <child link="${prefix}right_wheel"/>
+    <joint name="right_wheel_joint" type="continuous">
+      <parent link="base_link"/>
+      <child link="right_wheel"/>
       <origin xyz="0 ${-(base_width/2+wheel_yoff)} ${wheel_zoff}" rpy="${pi/2} 0 0"/>
       <axis xyz="0 0 -1"/>
@@ -88,5 +88,5 @@
     </joint>
     <!-- right wheel Link -->
-    <link name="${prefix}right_wheel">
+    <link name="right_wheel">
       <collision>
         <geometry>

Commit message: Added gazebo info and increased board B update rate

File: imprimis_ws/src/imprimis_description/urdf/diffbot.ros2_control.xacro (robot description, xacro)
@@ -1,7 +1,8 @@
 <?xml version="1.0"?>
 <robot xmlns:xacro="http://www.ros.org/wiki/xacro">
-  <xacro:macro name="diffbot_ros2_control" params="name use_mock_hardware">
+  <xacro:macro name="diffbot_ros2_control" params="name hardware_type">
     <ros2_control name="${name}" type="system">
-      <xacro:unless value="${use_mock_hardware}">
+    <!-- Real hardware -->
+      <xacro:if value="${hardware_type == 'real'}">
         <hardware>
           <plugin>imprimis_hardware_platform/DiffBotSystemHardware</plugin>
@@ -9,6 +10,7 @@
           <param name="example_param_hw_stop_duration_sec">3.0</param>
         </hardware>
-      </xacro:unless>
-      <xacro:if value="${use_mock_hardware}">
+      </xacro:if>
+    <!-- Fake hardware-->
+      <xacro:if value="${hardware_type == 'fake'}">
         <hardware>
           <plugin>mock_components/GenericSystem</plugin>
@@ -16,4 +18,12 @@
         </hardware>
       </xacro:if>
+    <!-- TODO gazebo-simulated Hardware -->
+      <xacro:if value="${hardware_type == 'simulated'}">
+        <hardware>
+          <plugin>mock_components/GenericSystem</plugin>
+          <param name="calculate_dynamics">true</param>
+        </hardware>
+      </xacro:if>
+    <!-- Joint definitions -->
       <joint name="left_wheel_joint">
         <command_interface name="velocity"/>

File: imprimis_ws/src/imprimis_description/urdf/diffbot.urdf.xacro (robot description, xacro)
@@ -2,12 +2,15 @@
 <!-- Basic differential drive mobile base -->
 <robot xmlns:xacro="http://www.ros.org/wiki/xacro" name="diffdrive_robot">
-  <xacro:arg name="use_mock_hardware" default="false" />
+  <xacro:arg name="hardware_type" default="real" />
+  <!-- Import and expand core robot description -->
   <xacro:include filename="$(find imprimis_description)/urdf/diffbot_description.urdf.xacro" />
+  <xacro:diffbot/>
   <!-- Import Rviz colors -->
   <xacro:include filename="$(find imprimis_description)/urdf/diffbot.materials.xacro" />
-  <!-- Import diffbot ros2_control description -->
+  <!-- Import and expand diffbot ros2_control description -->
   <xacro:include filename="$(find imprimis_description)/urdf/diffbot.ros2_control.xacro" />
-  <xacro:diffbot/>
-  <xacro:diffbot_ros2_control
-    name="DiffBot" use_mock_hardware="$(arg use_mock_hardware)"/>
+  <xacro:diffbot_ros2_control name="DiffBot" hardware_type="$(arg hardware_type)"/>
+  <!-- Import and expand gazebo information -->
+  <xacro:include filename="$(find imprimis_description)/urdf/gazebo_info.xacro"/>
+  <xacro:gazebo_info/>
 </robot>

Commit message: Added gazebo simulation and modified hardware launch file

File: imprimis_ws/src/imprimis_description/urdf/diffbot.ros2_control.xacro (robot description, xacro)
@@ -18,9 +18,8 @@
         </hardware>
       </xacro:if>
-    <!-- TODO gazebo-simulated Hardware -->
+    <!-- Gazebo-simulated Hardware -->
       <xacro:if value="${hardware_type == 'simulated'}">
         <hardware>
-          <plugin>mock_components/GenericSystem</plugin>
-          <param name="calculate_dynamics">true</param>
+          <plugin>gazebo_ros2_control/GazeboSystem</plugin>
         </hardware>
       </xacro:if>

File: imprimis_ws/src/imprimis_description/urdf/diffbot.urdf.xacro (robot description, xacro)
@@ -11,6 +11,5 @@
   <xacro:include filename="$(find imprimis_description)/urdf/diffbot.ros2_control.xacro" />
   <xacro:diffbot_ros2_control name="DiffBot" hardware_type="$(arg hardware_type)"/>
-  <!-- Import and expand gazebo information -->
+  <!-- Import gazebo information -->
   <xacro:include filename="$(find imprimis_description)/urdf/gazebo_info.xacro"/>
-  <xacro:gazebo_info/>
 </robot>

File: imprimis_ws/src/imprimis_description/urdf/diffbot_description.urdf.xacro (robot description, xacro)
@@ -2,5 +2,4 @@
 <robot xmlns:xacro="http://www.ros.org/wiki/xacro">
 <xacro:macro name="diffbot">
-<!-- Constants for robot dimensions -->
 <xacro:property name="PI" value="3.1415926535897931"/>
 <!-- Constants for robot dimensions -->
@@ -17,6 +16,8 @@
 <xacro:property name="base_top_height" value="0.305"/>
 <xacro:include filename="inertial_macros.xacro" />
+<!-- Base link -->
 <link name="base_link">
 </link>
+<!-- Base footprint joint and link -->
 <joint name="base_footprint_joint" type="fixed">
   <parent link="base_link"/>
@@ -26,4 +27,5 @@
 <link name="base_footprint">
 </link>
+<!-- Chassis joint -->
 <joint name="chassis_joint" type="fixed">
   <parent link="base_link"/>
@@ -31,4 +33,5 @@
   <origin xyz="-0.85 0 0"/>
 </joint>
+<!-- Chassis link -->
 <link name="chassis">
   <visual>
@@ -49,4 +52,5 @@
   </xacro:inertial_box>
 </link>
+<!-- Left wheel joint -->
 <joint name="left_wheel_joint" type="continuous">
   <parent link="base_link"/>
@@ -56,5 +60,5 @@
   <dynamics damping="0.2"/>
 </joint>
-    <!-- left wheel Link -->
+<!-- Left wheel Link -->
 <link name="left_wheel">
   <collision>
@@ -80,12 +84,13 @@
     </inertial>
   </link>
-    <joint name="right_wheel_joint" type="continuous">
-      <parent link="base_link"/>
-      <child link="right_wheel"/>
-      <origin xyz="0 ${-(base_width/2+wheel_yoff)} ${wheel_zoff}" rpy="${pi/2} 0 0"/>
-      <axis xyz="0 0 -1"/>
-      <dynamics damping="0.1"/>
-    </joint>
-    <!-- right wheel Link -->
+  <!-- Right wheel joint -->
+  <joint name="right_wheel_joint" type="continuous">
+    <parent link="base_link"/>
+    <child link="right_wheel"/>
+    <origin xyz="0 ${-(base_width/2+wheel_yoff)} ${wheel_zoff}" rpy="${pi/2} 0 0"/>
+    <axis xyz="0 0 -1"/>
+    <dynamics damping="0.1"/>
+  </joint>
+    <!-- Right wheel Link -->
     <link name="right_wheel">
       <collision>

File: imprimis_ws/src/imprimis_description/urdf/gazebo_info.xacro (robot description, xacro)
@@ -1,5 +1,24 @@
 <?xml version="1.0"?>
 <robot xmlns:xacro="http://www.ros.org/wiki/xacro">
-  <xacro:macro name="gazebo_info">
-  </xacro:macro>
+  <!-- Make the wheels black -->
+  <gazebo reference="left_wheel">
+    <material>Gazebo/Black</material>
+  </gazebo>
+  <gazebo reference="right_wheel">
+    <material>Gazebo/Black</material>
+  </gazebo>
+  <!-- This will publish the joint states of the wheels in the simulation-->
+  <gazebo>
+    <plugin name="gazebo_ros_joint_state_publisher" filename="libgazebo_ros_joint_state_publisher.so">
+      <update_rate>50</update_rate>
+      <joint_name>left_wheel_joint</joint_name>
+      <joint_name>right_wheel_joint</joint_name>
+    </plugin>
+  </gazebo>
+  <!-- This is the ros2 control gazebo plugin -->
+  <gazebo>
+    <plugin name="gazebo_ros2_control" filename="libgazebo_ros2_control.so">
+      <parameters>$(find imprimis_hardware_platform)/config/sim_diffbot_controllers.yaml</parameters>
+    </plugin>
+  </gazebo>
 </robot>

Commit message: Upgraded gazebo simulation

File: imprimis_ws/src/imprimis_description/urdf/diffbot.ros2_control.xacro (robot description, xacro)
@@ -21,5 +21,5 @@
       <xacro:if value="${hardware_type == 'simulated'}">
         <hardware>
-          <plugin>gazebo_ros2_control/GazeboSystem</plugin>
+          <plugin>gz_ros2_control/GazeboSimSystem</plugin>
         </hardware>
       </xacro:if>

File: imprimis_ws/src/imprimis_description/urdf/diffbot.urdf.xacro (robot description, xacro)
@@ -11,5 +11,6 @@
   <xacro:include filename="$(find imprimis_description)/urdf/diffbot.ros2_control.xacro" />
   <xacro:diffbot_ros2_control name="DiffBot" hardware_type="$(arg hardware_type)"/>
-  <!-- Import gazebo information -->
+  <!-- Import and expand gazebo information. It's fine to keep it in there even if hardware type isn't simulated. -->
   <xacro:include filename="$(find imprimis_description)/urdf/gazebo_info.xacro"/>
+  <xacro:gzinfo/>
 </robot>

File: imprimis_ws/src/imprimis_description/urdf/diffbot_description.urdf.xacro (robot description, xacro)
@@ -193,8 +193,8 @@
 </link>
 <!-- Lidar joint and link -->
-<xacro:include filename="$(find velodyne_description)/urdf/VLP-16.urdf.xacro"/>
+<!--xacro:include filename="$(find velodyne_description)/urdf/VLP-16.urdf.xacro"/>
   <xacro:VLP-16 parent="lidar_pole" name="velodyne" topic="/velodyne_points" organize_cloud="false" hz="10" samples="440" gpu="false">
     <origin xyz="0 0 ${lidar_pole_height}" rpy="0 ${lidar_pole_angle} 0" />
-  </xacro:VLP-16>
+  </xacro:VLP-16-->
 </xacro:macro>
 </robot>

File: imprimis_ws/src/imprimis_description/urdf/gazebo_info.xacro (robot description, xacro)
@@ -1,4 +1,5 @@
 <?xml version="1.0"?>
 <robot xmlns:xacro="http://www.ros.org/wiki/xacro">
+<xacro:macro name="gzinfo">
   <!-- Make the wheels black and have lots of friction -->
   <gazebo reference="left_wheel">
@@ -22,17 +23,30 @@
     <material>Gazebo/Gray</material>
   </gazebo>
-  <!-- This will publish the joint states of the wheels in the simulation-->
   <gazebo>
-    <plugin name="gazebo_ros_joint_state_publisher" filename="libgazebo_ros_joint_state_publisher.so">
-      <update_rate>50</update_rate>
+    <!-- Joint state publisher plugin-->
+    <plugin filename="gz-sim-joint-state-publisher-system" name="gz::sim::systems::JointStatePublisher">
+      <topic>joint_states</topic>
       <joint_name>left_wheel_joint</joint_name>
       <joint_name>right_wheel_joint</joint_name>
     </plugin>
+  <!-- ros2 control plugin -->
+  <plugin name="gz_ros2_control::GazeboSimROS2ControlPlugin" filename="gz_ros2_control-system">
+    <parameters>$(find imprimis_hardware_platform)/config/sim_diffbot_controllers.yaml</parameters>
+  </plugin>
+    <!-- Diff drive controller plugin>
+    <plugin name="gz::sim::systems::DiffDrive" filename="gz-sim-diff-drive-system">
+      <left_joint>left_wheel_joint</left_joint>
+      <right_joint>right_wheel_joint</right_joint>
+      <wheel_separation>1.016</wheel_separation>
+      <wheel_radius>0.165</wheel_radius>
+      <max_linear_acceleration>1.5</max_linear_acceleration>
+      <topic>diffbot_base_controller/cmd_vel</topic>
+      <frame_id>odom</frame_id>
+      <child_frame_id>base_link</child_frame_id>
+      <odom_topic>diffbot_base_controller/odom</odom_topic>
+      <odom_publisher_frequency>30</odom_publisher_frequency>
+      <tf_topic>/tf</tf_topic>
+    </plugin-->
   </gazebo>
-  <!-- This is the ros2 control gazebo plugin -->
-  <gazebo>
-    <plugin name="gazebo_ros2_control" filename="libgazebo_ros2_control.so">
-      <parameters>$(find imprimis_hardware_platform)/config/sim_diffbot_controllers.yaml</parameters>
-    </plugin>
-  </gazebo>
+  </xacro:macro>
 </robot>
