Commit message: Added GPS and noise to IMU, and publish odom tf option for simulation

File: imprimis_ws/src/imprimis_description/urdf/diffbot.urdf.xacro (robot description, xacro)
@@ -3,4 +3,5 @@
 <robot xmlns:xacro="http://www.ros.org/wiki/xacro" name="diffdrive_robot">
   <xacro:arg name="hardware_type" default="real" />
+  <xacro:arg name="publish_odom_tf" default="true" />
   <!-- Import and expand core robot description -->
   <xacro:include filename="$(find imprimis_description)/urdf/diffbot_description.urdf.xacro" />
@@ -13,4 +14,4 @@
   <!-- Import and expand gazebo information. It's fine to keep it in there even if hardware type isn't simulated. -->
   <xacro:include filename="$(find imprimis_description)/urdf/gazebo_info.xacro"/>
-  <xacro:gzinfo/>
+  <xacro:gzinfo publish_odom_tf="$(arg publish_odom_tf)"/>
 </robot>

File: imprimis_ws/src/imprimis_description/urdf/diffbot_description.urdf.xacro (robot description, xacro)
@@ -214,10 +214,4 @@
     </geometry>
   </visual>
-  <collision>
-    <origin rpy="0 0 0" xyz="0 0 0.03585"/>
-    <geometry>
-      <cylinder radius="0.0516" length="0.0717"/>
-    </geometry>
-  </collision>
 </link>
 <!-- Lidar model joint -->

File: imprimis_ws/src/imprimis_description/urdf/gazebo_info.xacro (robot description, xacro)
@@ -1,5 +1,5 @@
 <?xml version="1.0"?>
 <robot xmlns:xacro="http://www.ros.org/wiki/xacro">
-<xacro:macro name="gzinfo">
+<xacro:macro name="gzinfo" params="publish_odom_tf">
   <!-- Make the wheels black and have lots of friction -->
   <gazebo reference="left_wheel">
@@ -49,9 +49,9 @@
         <max>100.0</max>
         <resolution>0.01</resolution>
+        <!--noise type="gaussian">
+          <mean>0.0</mean>
+          <stddev>0.01</stddev>
+        </noise-->
       </range>
-      <!--noise type="gaussian">
-        <mean>0.0</mean>
-        <stddev>0.01</stddev>
-      </noise-->
     </ray>
     <always_on>true</always_on>
@@ -66,5 +66,37 @@
     <update_rate>50</update_rate>
     <always_on>true</always_on>
-    <visualize>true</visualize>
+    <imu>
+      <angular_velocity>
+        <noise type="gaussian">
+          <mean>0</mean>
+          <stddev>0.0002</stddev>
+        </noise>
+      </angular_velocity>
+      <linear_acceleration>
+        <noise type="gaussian">
+          <mean>0</mean>
+          <stddev>0.01</stddev>
+        </noise>
+      </linear_acceleration>
+    </imu>
+    </sensor>
+  </gazebo>
+  <!-- Simulated GPS configuration -->
+  <gazebo reference="gps_link">
+    <sensor name="gps_sensor" type="navsat">
+    <pose> 0 0 0 0 0 0 </pose>
+    <topic>gps</topic>
+    <update_rate>5</update_rate>
+    <always_on>true</always_on>
+    <navsat>
+      <position_sensing>
+        <horizontal>
+          <noise type="gaussian">
+            <mean>0</mean>
+            <stddev>1.5</stddev>  <!-- meters -->
+          </noise>
+        </horizontal>
+      </position_sensing>
+    </navsat>
     </sensor>
   </gazebo>
@@ -79,4 +111,7 @@
   <plugin name="gz_ros2_control::GazeboSimROS2ControlPlugin" filename="gz_ros2_control-system">
     <parameters>$(find imprimis_hardware_platform)/config/sim_diffbot_controllers.yaml</parameters>
+    <xacro:unless value="${publish_odom_tf}">
+      <parameters>$(find imprimis_hardware_platform)/config/disable_odom_tf.yaml</parameters>
+    </xacro:unless>
   </plugin>
   <!-- Simulated sensor manager plugin -->
@@ -87,4 +122,5 @@
   <plugin filename="libignition-gazebo-imu-system.so" name="ignition::gazebo::systems::Imu"/>
   <!-- GPS sensor plugin -->
+  <plugin filename="libignition-gazebo-navsat-system.so" name="ignition::gazebo::systems::NavSat"/>
   </gazebo>
   </xacro:macro>
