Commit message: Modified robot URDF and gazebo parameters

File: imprimis_ws/src/imprimis_description/urdf/diffbot_description.urdf.xacro (robot description, xacro)
@@ -4,5 +4,5 @@
 <xacro:property name="PI" value="3.1415926535897931"/>
 <!-- Constants for robot dimensions -->
-<xacro:property name="base_mass" value="0.3" />
+<xacro:property name="base_mass" value="30.0" />
 <xacro:property name="wheel_mass" value="0.3" />
 <xacro:property name="base_width" value="0.62" />
@@ -15,4 +15,12 @@
 <xacro:property name="base_top_width" value="0.749"/>
 <xacro:property name="base_top_height" value="0.305"/>
+<xacro:property name="lidar_pole_side" value="0.025"/> <!-- TODO measure lidar pole values -->
+<xacro:property name="lidar_pole_height" value="1.0"/>
+<xacro:property name="lidar_pole_xoff" value="0.5"/>
+<xacro:property name="lidar_pole_mass" value="2.0"/>
+<!-- Constants for simulated caster wheel-->
+<xacro:property name="caster_mass" value="0.1"/>
+<xacro:property name="caster_radius" value="0.105"/>
+<xacro:property name="caster_xoff" value="0.15"/>
 <xacro:include filename="inertial_macros.xacro" />
 <!-- Base link -->
@@ -48,5 +56,5 @@
     </geometry>
   </collision>
-  <xacro:inertial_box mass="0.5" x="${base_length}" y="${base_width}" z="${base_height}"> <!-- inertial macro -->
+  <xacro:inertial_box mass="${base_mass}" x="${base_length}" y="${base_width}" z="${base_height}"> <!-- inertial macro -->
     <origin xyz="${base_length/2} 0 ${base_height/2}" rpy="0 0 0"/>
   </xacro:inertial_box>
@@ -58,5 +66,5 @@
   <origin xyz="0 ${base_width/2+wheel_yoff} ${wheel_zoff}" rpy="-${pi/2} 0 0"/>
   <axis xyz="0 0 1"/>
-  <dynamics damping="0.2"/>
+  <dynamics damping="0.0"/>
 </joint>
 <!-- Left wheel Link -->
@@ -82,36 +90,83 @@
       iyy="${wheel_mass / 12.0 * (3*wheel_radius*wheel_radius + wheel_len*wheel_len)}" iyz="0.0"
       izz="${wheel_mass / 2.0 * wheel_radius*wheel_radius}"/>
-    </inertial>
-  </link>
-  <!-- Right wheel joint -->
-  <joint name="right_wheel_joint" type="continuous">
-    <parent link="base_link"/>
-    <child link="right_wheel"/>
-    <origin xyz="0 ${-(base_width/2+wheel_yoff)} ${wheel_zoff}" rpy="${pi/2} 0 0"/>
-    <axis xyz="0 0 -1"/>
-    <dynamics damping="0.1"/>
-  </joint>
-    <!-- Right wheel Link -->
-    <link name="right_wheel">
-      <collision>
-        <geometry>
-          <cylinder length="${wheel_len}" radius="${wheel_radius}"/>
-        </geometry>
-      </collision>
-      <visual>
-        <geometry>
-          <cylinder length="${wheel_len}" radius="${wheel_radius}"/>
-        </geometry>
-        <material name="black"/>
-      </visual>
-      <inertial>
-        <origin xyz="0 0 0" rpy="${PI/2} 0 0"/>
-        <mass value="${wheel_mass}"/>
-        <inertia
-          ixx="${wheel_mass / 12.0 * (3*wheel_radius*wheel_radius + wheel_len*wheel_len)}" ixy="0.0" ixz="0.0"
-          iyy="${wheel_mass / 12.0 * (3*wheel_radius*wheel_radius + wheel_len*wheel_len)}" iyz="0.0"
-          izz="${wheel_mass / 2.0 * wheel_radius*wheel_radius}"/>
-        </inertial> <!-- for some reason, the inertial cylinder macro was not parsing -->
-      </link>
-  </xacro:macro>
+  </inertial>
+</link>
+<!-- Right wheel joint -->
+<joint name="right_wheel_joint" type="continuous">
+  <parent link="base_link"/>
+  <child link="right_wheel"/>
+  <origin xyz="0 ${-(base_width/2+wheel_yoff)} ${wheel_zoff}" rpy="${pi/2} 0 0"/>
+  <axis xyz="0 0 -1"/>
+  <dynamics damping="0.0"/>
+</joint>
+<!-- Right wheel Link -->
+<link name="right_wheel">
+  <collision>
+    <geometry>
+      <cylinder length="${wheel_len}" radius="${wheel_radius}"/>
+    </geometry>
+  </collision>
+  <visual>
+    <geometry>
+      <cylinder length="${wheel_len}" radius="${wheel_radius}"/>
+    </geometry>
+    <material name="black"/>
+  </visual>
+  <inertial>
+    <origin xyz="0 0 0" rpy="${PI/2} 0 0"/>
+    <mass value="${wheel_mass}"/>
+    <inertia
+      ixx="${wheel_mass / 12.0 * (3*wheel_radius*wheel_radius + wheel_len*wheel_len)}" ixy="0.0" ixz="0.0"
+      iyy="${wheel_mass / 12.0 * (3*wheel_radius*wheel_radius + wheel_len*wheel_len)}" iyz="0.0"
+      izz="${wheel_mass / 2.0 * wheel_radius*wheel_radius}"/>
+  </inertial> <!-- for some reason, the inertial cylinder macro was not parsing -->
+</link>
+  <!-- Caster joint -->
+<joint name="caster_joint" type="fixed">
+  <parent link="chassis"/>
+  <child link="caster_sphere"/>
+  <origin xyz="${caster_xoff} 0 0"/>
+</joint>
+<!-- Caster link -->
+<link name="caster_sphere">
+  <visual>
+    <geometry>
+      <sphere radius="${caster_radius}"/>
+    </geometry>
+  <material name="white"/>
+  </visual>
+  <collision>
+    <geometry>
+      <sphere radius="${caster_radius}"/>
+    </geometry>
+  </collision>
+  <inertial>
+    <mass value="${caster_mass}" />
+    <inertia ixx="${(2/5) * caster_mass * (caster_radius*caster_radius)}" ixy="0.0" ixz="0.0"
+            iyy="${(2/5) * caster_mass * (caster_radius*caster_radius)}" iyz="0.0"
+            izz="${(2/5) * caster_mass * (caster_radius*caster_radius)}" />
+  </inertial>
+</link>
+<joint name="lidar_pole_joint" type="fixed">
+  <parent link="chassis"/>
+  <child link="lidar_pole"/>
+  <origin xyz="${lidar_pole_xoff} 0 ${base_height}"/>
+</joint>
+<link name="lidar_pole">
+  <visual>
+    <geometry>
+      <box size="${lidar_pole_side} ${lidar_pole_side} ${lidar_pole_height}"/>
+    </geometry>
+  <material name="grey"/>
+  </visual>
+  <collision>
+    <geometry>
+      <box size="${lidar_pole_side} ${lidar_pole_side} ${lidar_pole_height}"/>
+    </geometry>
+  </collision>
+  <xacro:inertial_box mass="${lidar_pole_mass}" x="${lidar_pole_side}" y="${lidar_pole_side}" z="${lidar_pole_height}"> <!-- inertial macro -->
+    <origin xyz="0 0 0" rpy="0 0 0"/>
+  </xacro:inertial_box>
+</link>
+</xacro:macro>
 </robot>

File: imprimis_ws/src/imprimis_description/urdf/gazebo_info.xacro (robot description, xacro)
@@ -1,10 +1,24 @@
 <?xml version="1.0"?>
 <robot xmlns:xacro="http://www.ros.org/wiki/xacro">
-  <!-- Make the wheels black -->
+  <!-- Make the wheels black and have lots of friction -->
   <gazebo reference="left_wheel">
     <material>Gazebo/Black</material>
+    <mu1 value="6.0"/>
+    <mu2 value="6.0"/>
   </gazebo>
   <gazebo reference="right_wheel">
     <material>Gazebo/Black</material>
+    <mu1 value="6.0"/>
+    <mu2 value="6.0"/>
+  </gazebo>
+  <!-- Make the caster wheel white and have no friction -->
+  <gazebo reference="caster_sphere">
+    <material>Gazebo/White</material>
+    <mu1 value="0.0001"/>
+    <mu2 value="0.0001"/>
+  </gazebo>
+  <!-- Make the lidar pole gray-->
+  <gazebo reference="lidar_pole">
+    <material>Gazebo/Gray</material>
   </gazebo>
   <!-- This will publish the joint states of the wheels in the simulation-->

Commit message: Added simulated velodyne lidar to URDF

File: imprimis_ws/src/imprimis_description/urdf/diffbot_description.urdf.xacro (robot description, xacro)
@@ -148,4 +148,5 @@
   </inertial>
 </link>
+<!-- Lidar pole joint-->
 <joint name="lidar_pole_joint" type="fixed">
   <parent link="chassis"/>
@@ -153,4 +154,5 @@
   <origin xyz="${lidar_pole_xoff} 0 ${base_height}"/>
 </joint>
+<!-- Lidar pole link-->
 <link name="lidar_pole">
   <visual>
@@ -169,4 +171,9 @@
   </xacro:inertial_box>
 </link>
+<!-- Lidar joint and link -->
+<xacro:include filename="$(find velodyne_description)/urdf/VLP-16.urdf.xacro"/>
+  <xacro:VLP-16 parent="lidar_pole" name="velodyne" topic="/velodyne_points" organize_cloud="false" hz="10" samples="440" gpu="false">
+    <origin xyz="0 0 ${lidar_pole_height/2}" rpy="0 0 0" />
+  </xacro:VLP-16>
 </xacro:macro>
 </robot>

Commit message: Added nav_configs package and t265_ros_driver package.

File: imprimis_ws/src/imprimis_description/urdf/diffbot_description.urdf.xacro (robot description, xacro)
@@ -16,5 +16,5 @@
 <xacro:property name="base_top_height" value="0.305"/>
 <xacro:property name="lidar_pole_side" value="0.025"/> <!-- TODO measure lidar pole values -->
-<xacro:property name="lidar_pole_height" value="1.0"/>
+<xacro:property name="lidar_pole_height" value="0.6"/>
 <xacro:property name="lidar_pole_xoff" value="0.5"/>
 <xacro:property name="lidar_pole_mass" value="2.0"/>
@@ -152,5 +152,5 @@
   <parent link="chassis"/>
   <child link="lidar_pole"/>
-  <origin xyz="${lidar_pole_xoff} 0 ${base_height}"/>
+  <origin xyz="${lidar_pole_xoff} 0 ${(3/2) * base_height}"/>
 </joint>
 <!-- Lidar pole link-->

Commit message: Added t265, commented out lidar in launch file, fixed measurements in URDF

File: imprimis_ws/src/imprimis_description/urdf/diffbot_description.urdf.xacro (robot description, xacro)
@@ -15,8 +15,10 @@
 <xacro:property name="base_top_width" value="0.749"/>
 <xacro:property name="base_top_height" value="0.305"/>
-<xacro:property name="lidar_pole_side" value="0.025"/> <!-- TODO measure lidar pole values -->
-<xacro:property name="lidar_pole_height" value="0.6"/>
-<xacro:property name="lidar_pole_xoff" value="0.5"/>
+<xacro:property name="lidar_pole_side" value="0.023"/>
+<xacro:property name="lidar_pole_height" value="0.635"/> <!-- height from the top of chassis to lidar-->
+<xacro:property name="lidar_pole_xoff" value="0.48"/> <!-- length from back of robot to lidar pole-->
 <xacro:property name="lidar_pole_mass" value="2.0"/>
+<xacro:property name="t265_mount_zoff" value="0.421"/> <!-- height from top of chassis to the camera-->
+<xacro:property name="lidar_pole_angle" value="0.035"/> <!-- tilt of the lidar pole along the x axis-->
 <!-- Constants for simulated caster wheel-->
 <xacro:property name="caster_mass" value="0.1"/>
@@ -152,5 +154,5 @@
   <parent link="chassis"/>
   <child link="lidar_pole"/>
-  <origin xyz="${lidar_pole_xoff} 0 ${(3/2) * base_height}"/>
+  <origin xyz="${lidar_pole_xoff} 0 ${base_height}"/>
 </joint>
 <!-- Lidar pole link-->
@@ -161,4 +163,5 @@
     </geometry>
   <material name="grey"/>
+  <origin xyz="0 0 ${lidar_pole_height/2}"/>
   </visual>
   <collision>
@@ -166,13 +169,23 @@
       <box size="${lidar_pole_side} ${lidar_pole_side} ${lidar_pole_height}"/>
     </geometry>
+    <origin xyz="0 0 ${lidar_pole_height/2}"/>
   </collision>
   <xacro:inertial_box mass="${lidar_pole_mass}" x="${lidar_pole_side}" y="${lidar_pole_side}" z="${lidar_pole_height}"> <!-- inertial macro -->
-    <origin xyz="0 0 0" rpy="0 0 0"/>
+    <origin xyz="0 0 ${lidar_pole_height/2}" rpy="0 0 0"/>
   </xacro:inertial_box>
+</link>
+<!-- t265 joint-->
+<joint name="t265_joint" type="fixed">
+  <parent link="lidar_pole"/>
+  <child link="t265"/>
+  <origin xyz="0 0 ${t265_mount_zoff}"/>
+</joint>
+<!-- t265 link -->
+<link name="t265">
 </link>
 <!-- Lidar joint and link -->
 <xacro:include filename="$(find velodyne_description)/urdf/VLP-16.urdf.xacro"/>
   <xacro:VLP-16 parent="lidar_pole" name="velodyne" topic="/velodyne_points" organize_cloud="false" hz="10" samples="440" gpu="false">
-    <origin xyz="0 0 ${lidar_pole_height/2}" rpy="0 0 0" />
+    <origin xyz="0 0 ${lidar_pole_height}" rpy="0 0 0" />
   </xacro:VLP-16>
 </xacro:macro>

Commit message: Fixed lidar pole angle in URDF

File: imprimis_ws/src/imprimis_description/urdf/diffbot_description.urdf.xacro (robot description, xacro)
@@ -20,5 +20,5 @@
 <xacro:property name="lidar_pole_mass" value="2.0"/>
 <xacro:property name="t265_mount_zoff" value="0.421"/> <!-- height from top of chassis to the camera-->
-<xacro:property name="lidar_pole_angle" value="0.035"/> <!-- tilt of the lidar pole along the x axis-->
+<xacro:property name="lidar_pole_angle" value="0.033"/> <!-- slight tilt of the lidar pole along the x axis-->
 <!-- Constants for simulated caster wheel-->
 <xacro:property name="caster_mass" value="0.1"/>
@@ -154,5 +154,5 @@
   <parent link="chassis"/>
   <child link="lidar_pole"/>
-  <origin xyz="${lidar_pole_xoff} 0 ${base_height}"/>
+  <origin xyz="${lidar_pole_xoff} 0 ${base_height}" rpy="0 ${-lidar_pole_angle} 0"/>
 </joint>
 <!-- Lidar pole link-->
@@ -187,5 +187,5 @@
 <xacro:include filename="$(find velodyne_description)/urdf/VLP-16.urdf.xacro"/>
   <xacro:VLP-16 parent="lidar_pole" name="velodyne" topic="/velodyne_points" organize_cloud="false" hz="10" samples="440" gpu="false">
-    <origin xyz="0 0 ${lidar_pole_height}" rpy="0 0 0" />
+    <origin xyz="0 0 ${lidar_pole_height}" rpy="0 ${lidar_pole_angle} 0" />
   </xacro:VLP-16>
 </xacro:macro>

Commit message: Added um7 IMU support

File: imprimis_ws/src/imprimis_description/urdf/diffbot_description.urdf.xacro (robot description, xacro)
@@ -19,5 +19,4 @@
 <xacro:property name="lidar_pole_xoff" value="0.48"/> <!-- length from back of robot to lidar pole-->
 <xacro:property name="lidar_pole_mass" value="2.0"/>
-<xacro:property name="t265_mount_zoff" value="0.421"/> <!-- height from top of chassis to the camera-->
 <xacro:property name="lidar_pole_angle" value="0.033"/> <!-- slight tilt of the lidar pole along the x axis-->
 <!-- Constants for simulated caster wheel-->
@@ -175,12 +174,21 @@
   </xacro:inertial_box>
 </link>
-<!-- t265 joint-->
-<joint name="t265_joint" type="fixed">
-  <parent link="lidar_pole"/>
-  <child link="t265"/>
-  <origin xyz="0 0 ${t265_mount_zoff}"/>
-</joint>
-<!-- t265 link -->
-<link name="t265">
+<!-- imu joint-->
+<joint name="imu_joint" type="fixed">
+  <parent link="base_link"/>
+  <child link="imu_link"/>
+  <origin xyz="0 0 0" rpy="0 0 0"/>
+</joint>
+<!-- imu link -->
+<link name="imu_link">
+</link>
+<!-- gps joint-->
+<joint name="gps_joint" type="fixed">
+  <parent link="base_link"/>
+  <child link="gps_link"/>
+  <origin xyz="0 0 0"/>
+</joint>
+<!-- gps link -->
+<link name="gps_link">
 </link>
 <!-- Lidar joint and link -->

Commit message: Added velodyne LIDAR to simulation

File: imprimis_ws/src/imprimis_description/urdf/diffbot_description.urdf.xacro (robot description, xacro)
@@ -192,9 +192,61 @@
 <link name="gps_link">
 </link>
+<!-- Lidar model link-->
+<link name="lidar_model_link">
+  <inertial>
+    <mass value="0.83"/>
+    <origin xyz="0 0 0.03585"/>
+    <inertia ixx="${(0.83 * (3.0*0.0516*0.0516 + 0.0717*0.0717)) / 12.0}" ixy="0" ixz="0"
+      iyy="${(0.83 * (3.0*0.0516*0.0516 + 0.0717*0.0717)) / 12.0}" iyz="0"
+      izz="${0.5 * 0.83 * (0.0516*0.0516)}"/>
+  </inertial>
+  <visual>
+    <geometry>
+      <mesh filename="package://imprimis_description/meshes/VLP16_base_1.dae" />
+    </geometry>
+  </visual>
+  <visual>
+    <geometry>
+      <mesh filename="package://imprimis_description/meshes/VLP16_base_2.dae" />
+    </geometry>
+  </visual>
+  <collision>
+    <origin rpy="0 0 0" xyz="0 0 0.03585"/>
+    <geometry>
+      <cylinder radius="0.0516" length="0.0717"/>
+    </geometry>
+  </collision>
+</link>
+<!-- Lidar model joint -->
+<joint name="$lidar_model_joint" type="fixed">
+  <parent link="lidar_pole"/>
+  <child link="lidar_model_link"/>
+  <origin xyz="0 0 ${lidar_pole_height}" rpy="0 ${lidar_pole_angle} 0" />
+</joint>
+<!-- Lidar scan point link -->
+<link name="lidar_scan_link">
+  <inertial>
+    <mass value="0.01"/>
+    <origin xyz="0 0 0"/>
+    <inertia ixx="1e-7" ixy="0" ixz="0" iyy="1e-7" iyz="0" izz="1e-7"/>
+  </inertial>
+  <visual>
+    <origin xyz="0 0 -0.0377" />
+    <geometry>
+      <mesh filename="package://imprimis_description/meshes/VLP16_scan.dae" />
+    </geometry>
+  </visual>
+</link>
+<!-- Lidar scan point joint -->
+<joint name="lidar_scan_joint" type="fixed" >
+  <origin xyz="0 0 0.0377" rpy="0 0 0" />
+  <parent link="lidar_model_link" />
+  <child link="lidar_scan_link"/>
+</joint>
 <!-- Lidar joint and link -->
 <!--xacro:include filename="$(find velodyne_description)/urdf/VLP-16.urdf.xacro"/>
-  <xacro:VLP-16 parent="lidar_pole" name="velodyne" topic="/velodyne_points" organize_cloud="false" hz="10" samples="440" gpu="false">
-    <origin xyz="0 0 ${lidar_pole_height}" rpy="0 ${lidar_pole_angle} 0" />
-  </xacro:VLP-16-->
+<xacro:VLP-16 parent="lidar_pole" name="velodyne" topic="/velodyne_points" organize_cloud="false" hz="10" samples="440" gpu="false">
+  <origin xyz="0 0 ${lidar_pole_height}" rpy="0 ${lidar_pole_angle} 0" />
+</xacro:VLP-16-->
 </xacro:macro>
 </robot>

File: imprimis_ws/src/imprimis_description/urdf/gazebo_info.xacro (robot description, xacro)
@@ -23,4 +23,42 @@
     <material>Gazebo/Gray</material>
   </gazebo>
+  <!-- Simulated lidar configuration -->
+  <gazebo reference="lidar_scan_link">
+    <sensor name="vlp16" type="gpu_lidar">
+    <gz_frame_id>lidar_scan_link</gz_frame_id>
+    <pose>0 0 0 0 0 0</pose>
+    <topic>lidar</topic>
+    <update_rate>10</update_rate>
+    <ray>
+      <scan>
+        <horizontal>
+          <samples>1800</samples>
+          <resolution>1</resolution>
+          <min_angle>-3.141592653589793</min_angle>
+          <max_angle>3.141592653589793</max_angle>
+        </horizontal>
+        <vertical>
+          <samples>16</samples>
+          <resolution>1</resolution>
+          <min_angle>-0.2617993877991494</min_angle>  <!-- -15 deg -->
+          <max_angle>0.2617993877991494</max_angle>   <!-- +15 deg -->
+        </vertical>
+      </scan>
+      <range>
+        <min>0.3</min>
+        <max>100.0</max>
+        <resolution>0.01</resolution>
+      </range>
+      <!--
+      <noise type="gaussian">
+        <mean>0.0</mean>
+        <stddev>0.01</stddev>
+      </noise>
+      -->
+    </ray>
+    <always_on>true</always_on>
+    <visualize>true</visualize>
+  </sensor>
+  </gazebo>
   <gazebo>
     <!-- Joint state publisher plugin-->
@@ -34,18 +72,8 @@
     <parameters>$(find imprimis_hardware_platform)/config/sim_diffbot_controllers.yaml</parameters>
   </plugin>
-    <!-- Diff drive controller plugin>
-    <plugin name="gz::sim::systems::DiffDrive" filename="gz-sim-diff-drive-system">
-      <left_joint>left_wheel_joint</left_joint>
-      <right_joint>right_wheel_joint</right_joint>
-      <wheel_separation>1.016</wheel_separation>
-      <wheel_radius>0.165</wheel_radius>
-      <max_linear_acceleration>1.5</max_linear_acceleration>
-      <topic>diffbot_base_controller/cmd_vel</topic>
-      <frame_id>odom</frame_id>
-      <child_frame_id>base_link</child_frame_id>
-      <odom_topic>diffbot_base_controller/odom</odom_topic>
-      <odom_publisher_frequency>30</odom_publisher_frequency>
-      <tf_topic>/tf</tf_topic>
-    </plugin-->
+  <!-- Simulated sensors plugin -->
+  <plugin filename="libignition-gazebo-sensors-system.so" name="ignition::gazebo::systems::Sensors">
+    <render_engine>ogre</render_engine>
+  </plugin>
   </gazebo>
   </xacro:macro>

Commit message: Added simulated IMU and gazebo-fixing script

File: imprimis_ws/src/imprimis_description/urdf/diffbot_description.urdf.xacro (robot description, xacro)
@@ -182,4 +182,7 @@
 <!-- imu link -->
 <link name="imu_link">
+  <xacro:inertial_box mass="0.1" x="0" y="0" z="0">
+    <origin xyz="0 0 0" rpy="0 0 0"/>
+  </xacro:inertial_box>
 </link>
 <!-- gps joint-->

File: imprimis_ws/src/imprimis_description/urdf/gazebo_info.xacro (robot description, xacro)
@@ -50,14 +50,22 @@
         <resolution>0.01</resolution>
       </range>
-      <!--
-      <noise type="gaussian">
+      <!--noise type="gaussian">
         <mean>0.0</mean>
         <stddev>0.01</stddev>
-      </noise>
-      -->
+      </noise-->
     </ray>
     <always_on>true</always_on>
     <visualize>true</visualize>
-  </sensor>
+    </sensor>
+  </gazebo>
+  <!-- Simulated IMU configuration -->
+  <gazebo reference="imu_link">
+    <sensor name="imu_sensor" type="imu">
+    <pose> 0 0 0 0 0 0 </pose>
+    <topic>imu</topic>
+    <update_rate>50</update_rate>
+    <always_on>true</always_on>
+    <visualize>true</visualize>
+    </sensor>
   </gazebo>
   <gazebo>
@@ -72,8 +80,11 @@
     <parameters>$(find imprimis_hardware_platform)/config/sim_diffbot_controllers.yaml</parameters>
   </plugin>
-  <!-- Simulated sensors plugin -->
+  <!-- Simulated sensor manager plugin -->
   <plugin filename="libignition-gazebo-sensors-system.so" name="ignition::gazebo::systems::Sensors">
     <render_engine>ogre</render_engine>
   </plugin>
+  <!-- IMU sensor plugin -->
+  <plugin filename="libignition-gazebo-imu-system.so" name="ignition::gazebo::systems::Imu"/>
+  <!-- GPS sensor plugin -->
   </gazebo>
   </xacro:macro>

Commit message: Fixed LIDAR and changed scan link name to match what converter package expects

File: imprimis_ws/src/imprimis_description/urdf/diffbot_description.urdf.xacro (robot description, xacro)
@@ -222,5 +222,5 @@
 </joint>
 <!-- Lidar scan point link -->
-<link name="lidar_scan_link">
+<link name="velodyne"> <!-- Must match the fixed frame in the VLP16 converter config, which defaults to 'velodyne'-->
   <inertial>
     <mass value="0.01"/>
@@ -239,5 +239,5 @@
   <origin xyz="0 0 0.0377" rpy="0 0 0" />
   <parent link="lidar_model_link" />
-  <child link="lidar_scan_link"/>
+  <child link="velodyne"/>
 </joint>
 <!-- Lidar joint and link -->

File: imprimis_ws/src/imprimis_description/urdf/gazebo_info.xacro (robot description, xacro)
@@ -24,7 +24,7 @@
   </gazebo>
   <!-- Simulated lidar configuration -->
-  <gazebo reference="lidar_scan_link">
+  <gazebo reference="velodyne"> <!-- Must match the lidar scan point link in diffbot description -->
     <sensor name="vlp16" type="gpu_lidar">
-    <gz_frame_id>lidar_scan_link</gz_frame_id>
+    <gz_frame_id>velodyne</gz_frame_id> <!-- Must match the lidar scan point link in diffbot description-->
     <pose>0 0 0 0 0 0</pose>
     <topic>lidar</topic>
@@ -60,5 +60,5 @@
   </gazebo>
   <!-- Simulated IMU configuration -->
-  <gazebo reference="imu_link">
+  <gazebo reference="imu_link"> <!-- Must match the imu link in diffbot description -->
     <sensor name="imu_sensor" type="imu">
     <pose> 0 0 0 0 0 0 </pose>
@@ -83,5 +83,5 @@
   </gazebo>
   <!-- Simulated GPS configuration -->
-  <gazebo reference="gps_link">
+  <gazebo reference="gps_link"> <!-- Must match the gps link in diffbot description -->
     <sensor name="gps_sensor" type="navsat">
     <pose> 0 0 0 0 0 0 </pose>

Commit message: Changed all navigation to work in the odom frame, added a new node to convert map goals to odom goals and correct for odom drift. Added GPS-based global localization; fixed navsat transform and global EKF. Added new SmacHybrid_DWB_2 nav2 params file.

File: imprimis_ws/src/imprimis_description/urdf/diffbot_description.urdf.xacro (robot description, xacro)
@@ -188,5 +188,5 @@
 <!-- gps joint-->
 <joint name="gps_joint" type="fixed">
-  <parent link="base_link"/>
+  <parent link="base_footprint"/>
   <child link="gps_link"/>
   <origin xyz="0 0 0"/>

File: imprimis_ws/src/imprimis_description/urdf/gazebo_info.xacro (robot description, xacro)
@@ -96,5 +96,5 @@
           <noise type="gaussian">
             <mean>0</mean>
-            <stddev>1.5e-6</stddev>
+            <stddev>3.0e-6</stddev>
           </noise>
         </horizontal>
