Commit message: changed urdf to add camera

File: imprimis_ws/src/imprimis_description/urdf/diffbot_description.urdf.xacro (robot description, xacro)
@@ -273,10 +273,15 @@
   <child link="velodyne"/>
 </joint>
-<!-- Camera joint and link -->
+<!-- Camera joint and link  -->
 <xacro:include filename="$(find realsense2_description)/urdf/_d435i.urdf.xacro"/>
 <xacro:sensor_d435i parent="chassis" name="front">
-  <origin xyz="${base_length+0.01} 0 ${base_height-0.022}" rpy="0 0 0"/>
-  <!-- Camera is placed slightly off from where it's mounted without these magic numbers. -->
+  <origin xyz="${base_length+0.01} 0 ${base_height-0.022+0.065}" rpy="0 0.1047 0"/>
 </xacro:sensor_d435i>
+<!-- Connect camera link to the rest of the robot
+<joint name="front_camera_joint" type="fixed" >
+  <origin xyz="0 0 0.486" rpy="0 0 0" />
+  <parent link="base_link" />
+  <child link="camera_link"/>
+</joint> -->
 <!-- Lidar joint and link -->
 <!--xacro:include filename="$(find velodyne_description)/urdf/VLP-16.urdf.xacro"/>

Commit message: added some performance upgrades and bug fixing to lane detection node, added dynamic camera angle and height

File: imprimis_ws/src/imprimis_description/urdf/diffbot_description.urdf.xacro (robot description, xacro)
@@ -276,5 +276,5 @@
 <xacro:include filename="$(find realsense2_description)/urdf/_d435i.urdf.xacro"/>
 <xacro:sensor_d435i parent="chassis" name="front">
-  <origin xyz="${base_length+0.01} 0 ${base_height-0.022+0.065}" rpy="0 0.1047 0"/>
+  <origin xyz="${base_length+0.01} 0 ${base_height-0.022+0.065}" rpy="0 0.2269 0"/>
 </xacro:sensor_d435i>
 <!-- Connect camera link to the rest of the robot

Commit message: Added julian's changes

File: imprimis_ws/src/imprimis_description/urdf/diffbot_description.urdf.xacro (robot description, xacro)
@@ -23,12 +23,22 @@
 <xacro:property name="lidar_pole_xoff" value="0.483"/>   <!-- 19.000" --> <!-- Back of robot to center of lidar pole-->
 <xacro:property name="lidar_pole_angle" value="0.033"/>                   <!-- Slight tilt of the lidar pole along the x-axis-->
-<xacro:property name="top_section_length" value="0.75"/> <!-- 25.560" --> <!-- Back of the robot to the end of the top section -->
+<xacro:property name="top_section_length" value="0.711"/> <!-- 28.000" --> <!-- Back of the robot to the end of the top section. Was 0.75 with a 25.56" comment; 0.711 is the SolidWorks value (Top_Panel_Glass). VERIFY WITH A TAPE MEASURE. -->
 <!-- Top section width is the same as base_width -->
 <xacro:property name="top_section_height" value="0.279"/> <!-- 11.000" --> <!-- Top of middle plane to top of top plane-->
 <!-- TOTAL ROBOT HEIGHT: 1.1173 m-->
-<!-- Simulated caster wheel-->
+<!-- Simulated caster wheels: two swivel casters at the rear corners, as on the real robot.
+     Positions are from the SolidWorks assembly HyperLabs Robot(07-03-25). Each is a low-friction
+     sphere whose lowest point touches the ground, so the deck sits level. -->
+<!-- Outline of the whole robot seen from above, measured from base_link (the drive axle).
+     The Nav2 footprint in config/nav2/FullFootprint.yaml must match these numbers.
+     Front edge +0.215 m (wheel_radius plus the camera). Rear edge -0.842 m (base_length minus wheel_radius).
+     Half width 0.486 m at the outer face of the tires (base_width/2 + wheel_yoff + wheel_len/2).
+     KEEP THESE COMMENTS DIRECTLY ABOVE AN XACRO TAG AND FREE OF COLONS. A comment that reaches the
+     generated URDF with a colon in it stops the launch (robot_description fails to parse as YAML). -->
 <xacro:property name="caster_mass" value="0.1"/>
-<xacro:property name="caster_radius" value="${wheel_radius - wheel_zoff}"/>
-<xacro:property name="caster_xoff" value="0.15"/>
+<xacro:property name="caster_radius" value="0.0445"/>  <!-- 03.500" diameter wheel -->
+<xacro:property name="caster_xoff" value="0.07"/>      <!-- 02.750" --> <!-- Back of robot to caster wheel center -->
+<xacro:property name="caster_yoff" value="0.272"/>     <!-- 10.700" --> <!-- Robot centerline to caster wheel center -->
+<xacro:property name="caster_zoff" value="${-(wheel_radius - wheel_zoff) + caster_radius}"/> <!-- Top of bottom plane down to caster center -->
 <!-- ***BEGIN ROBOT DESCRIPTION*** -->
 <!-- Base link -->
@@ -130,12 +140,38 @@
   </inertial> <!-- for some reason, the inertial cylinder macro was not parsing -->
 </link>
-  <!-- Caster joint -->
-<joint name="caster_joint" type="fixed">
+<!-- Left caster joint -->
+<joint name="caster_left_joint" type="fixed">
   <parent link="chassis"/>
-  <child link="caster_sphere"/>
-  <origin xyz="${caster_xoff} 0 0"/>
-</joint>
-<!-- Caster link -->
-<link name="caster_sphere">
+  <child link="caster_left"/>
+  <origin xyz="${caster_xoff} ${caster_yoff} ${caster_zoff}"/>
+</joint>
+<!-- Left caster link -->
+<link name="caster_left">
+  <visual>
+    <geometry>
+      <sphere radius="${caster_radius}"/>
+    </geometry>
+    <material name="white"/>
+  </visual>
+  <collision>
+    <geometry>
+      <sphere radius="${caster_radius}"/>
+    </geometry>
+  </collision>
+  <inertial>
+    <mass value="${caster_mass}" />
+    <inertia ixx="${(2/5) * caster_mass * (caster_radius*caster_radius)}" ixy="0.0" ixz="0.0"
+            iyy="${(2/5) * caster_mass * (caster_radius*caster_radius)}" iyz="0.0"
+            izz="${(2/5) * caster_mass * (caster_radius*caster_radius)}" />
+  </inertial>
+</link>
+<!-- Right caster joint -->
+<joint name="caster_right_joint" type="fixed">
+  <parent link="chassis"/>
+  <child link="caster_right"/>
+  <origin xyz="${caster_xoff} ${-caster_yoff} ${caster_zoff}"/>
+</joint>
+<!-- Right caster link -->
+<link name="caster_right">
   <visual>
     <geometry>
@@ -284,4 +320,33 @@
   <child link="camera_link"/>
 </joint> -->
+<!-- View camera for the IMPRIMIS Control window, on a pan and tilt head.
+     It is a simulator aid and not a part of the real robot. Navigation does not use it.
+     The head stands on the front edge of the top section, 0.97 m above the ground.
+     Pan turns without limit. Tilt is limited to a quarter circle up and a quarter circle down.
+     Positive tilt looks down. The links have no shape, so the LiDAR does not see them. -->
+<joint name="view_pan_joint" type="continuous">
+  <parent link="chassis"/>
+  <child link="view_pan"/>
+  <origin xyz="${top_section_length + 0.02} 0 ${base_height + top_section_height + 0.08}" rpy="0 0 0"/>
+  <axis xyz="0 0 1"/>
+  <limit effort="5.0" velocity="20.0"/>
+</joint>
+<link name="view_pan">
+  <xacro:inertial_sphere mass="0.02" radius="0.02">
+    <origin xyz="0 0 0" rpy="0 0 0"/>
+  </xacro:inertial_sphere>
+</link>
+<joint name="view_tilt_joint" type="revolute">
+  <parent link="view_pan"/>
+  <child link="view_camera"/>
+  <origin xyz="0 0 0" rpy="0 0 0"/>
+  <axis xyz="0 1 0"/>
+  <limit lower="-1.5708" upper="1.5708" effort="5.0" velocity="20.0"/>
+</joint>
+<link name="view_camera">
+  <xacro:inertial_sphere mass="0.02" radius="0.02">
+    <origin xyz="0 0 0" rpy="0 0 0"/>
+  </xacro:inertial_sphere>
+</link>
 <!-- Lidar joint and link -->
 <!--xacro:include filename="$(find velodyne_description)/urdf/VLP-16.urdf.xacro"/>

File: imprimis_ws/src/imprimis_description/urdf/gazebo_info.xacro (robot description, xacro)
@@ -13,6 +13,11 @@
     <mu2 value="6.0"/>
   </gazebo>
-  <!-- Make the caster wheel white and have no friction -->
-  <gazebo reference="caster_sphere">
+  <!-- Make the caster wheels white and have no friction -->
+  <gazebo reference="caster_left">
+    <material>Gazebo/White</material>
+    <mu1 value="0.0001"/>
+    <mu2 value="0.0001"/>
+  </gazebo>
+  <gazebo reference="caster_right">
     <material>Gazebo/White</material>
     <mu1 value="0.0001"/>
@@ -151,4 +156,24 @@
   </sensor>
 </gazebo>
+<!-- View camera of the IMPRIMIS Control window. It sees 60 m, where the front camera sees 10 m. -->
+<gazebo reference="view_camera">
+  <sensor name="view_rgb_camera" type="camera">
+    <gz_frame_id>view_camera</gz_frame_id>
+    <topic>/cameras/view/gzrgb/image_raw</topic>
+    <update_rate>20</update_rate>
+    <camera>
+      <horizontal_fov>1.52</horizontal_fov>
+      <image>
+        <width>960</width>
+        <height>540</height>
+        <format>R8G8B8</format>
+      </image>
+      <clip>
+        <near>0.05</near>
+        <far>60.0</far>
+      </clip>
+    </camera>
+  </sensor>
+</gazebo>
   <gazebo>
     <!-- Joint state publisher plugin-->
@@ -157,4 +182,23 @@
       <joint_name>left_wheel_joint</joint_name>
       <joint_name>right_wheel_joint</joint_name>
+      <joint_name>view_pan_joint</joint_name>
+      <joint_name>view_tilt_joint</joint_name>
+    </plugin>
+    <!-- Pan and tilt of the view camera. The angle wanted arrives on a topic and the joint is moved
+         to it by velocity, at up to 12 rad/s, so the tiny links need no tuning. -->
+    <plugin filename="gz-sim-joint-position-controller-system" name="gz::sim::systems::JointPositionController">
+      <joint_name>view_pan_joint</joint_name>
+      <topic>/view/pan_cmd</topic>
+      <use_velocity_commands>true</use_velocity_commands>
+      <cmd_max>12.0</cmd_max>
+      <cmd_min>-12.0</cmd_min>
+    </plugin>
+    <plugin filename="gz-sim-joint-position-controller-system" name="gz::sim::systems::JointPositionController">
+      <joint_name>view_tilt_joint</joint_name>
+      <topic>/view/tilt_cmd</topic>
+      <use_velocity_commands>true</use_velocity_commands>
+      <cmd_max>12.0</cmd_max>
+      <cmd_min>-12.0</cmd_min>
+      <initial_position>0.2</initial_position>
     </plugin>
   <!-- ros2 control plugin -->

Commit message: Significant improvement to ESP firmware, added nav perception launch file

File: imprimis_ws/src/imprimis_description/urdf/diffbot_description.urdf.xacro (robot description, xacro)
@@ -26,4 +26,5 @@
 <!-- Top section width is the same as base_width -->
 <xacro:property name="top_section_height" value="0.279"/> <!-- 11.000" --> <!-- Top of middle plane to top of top plane-->
+<xacro:property name="lidar_scan_angle" value="0.05"/>
 <!-- TOTAL ROBOT HEIGHT: 1.1173 m-->
 <!-- Simulated caster wheels: two swivel casters at the rear corners, as on the real robot.
@@ -305,5 +306,5 @@
 <!-- Lidar scan point joint -->
 <joint name="lidar_scan_joint" type="fixed" >
-  <origin xyz="0 0 0.0377" rpy="0 0 0" />
+  <origin xyz="0 0 0.0377" rpy="0 0 ${-lidar_scan_angle}" />
   <parent link="lidar_model_link" />
   <child link="velodyne"/>
